File: Stepped_Tone_Generator/Stepped_Tone_Generator.kicad_sch (KiCad schematic)
At the start: 19 parts, among them J1 FCV, J2 PWCV, J3 DC IN, J4 Audio Out, SW2 ON/OFF, U1 555, U2 555

Commit message: atari king layouts
Parts:
- R4: value 100K -> 10K
- R5: value 100K -> 4.7K
Connections:
- net PWR: now also FREQ1.3, PULSEWIDTH1.3; no longer R2.2, R3.2
- net at PULSEWIDTH1.2, U2.7 (DIS): now also R3.2; no longer R3.1
- net at FREQ1.2, U1.7 (DIS): now also R2.2; no longer R2.1
- net at C2.2, PULSEWIDTH1.1: no longer U2.6 (THR)
- net at C1.2, FREQ1.1, U1.2 (TR): no longer U1.6 (THR)
- new net: R3.1, U2.6 (THR)
- new net: R2.1, U1.6 (THR)
- no-connect marks 2 -> 0
Other:
- moved on the sheet: C2, PULSEWIDTH1
